File: hardware/emmc.kicad_sch (KiCad schematic)
At the start: 26 parts, among them U7 EMMC16G-TB29-PZ90, U9 MPFS025T-FCVG484E

Commit message: adding footprints to resistors and capacitors
Parts:
- R79: value R_US -> 0R; footprint (none) -> payload_footprints:RC0402N_YAG
Changed lines of the file:
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@@
 			)
 		)
-		(property "Value" "R_US"
+		(property "Value" "0R"
 			(at 106.934 97.79 90)
 			(show_name no)
@@
 			)
 		)
-		(property "Footprint" ""
+		(property "Footprint" "payload_footprints:RC0402N_YAG"
 			(at 101.854 98.044 90)
 			(hide yes)

Commit message: assigned footprints of resistors and some capacitors
Parts:
- C60, C61, C62, C63, C64, C65, C66, C67, C86, C87: value C -> 100nF; footprint (none) -> payload_footprints:CAPC1005X55N
- C85, C88: value C -> 4.7uF; footprint (none) -> payload_footprints:CAPC1608X90N
- R80, R81, R82: value R_US -> 10K; footprint (none) -> payload_footprints:RC0402N_YAG
- R83, R84, R85, R86, R87, R88, R89, R90: value R_US -> 49.9K; footprint (none) -> payload_footprints:RESC1005X40N
Changed lines of the file:
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@@
 			)
 		)
-		(property "Value" "R_US"
+		(property "Value" "49.9K"
 			(at 118.11 66.0399 0)
 			(show_name no)
@@
 			)
 		)
-		(property "Footprint" ""
+		(property "Footprint" "payload_footprints:RESC1005X40N"
 			(at 116.586 65.024 90)
 			(hide yes)
@@
 			)
 		)
-		(property "Value" "R_US"
+		(property "Value" "49.9K"
 			(at 90.17 66.0399 0)
 			(show_name no)
@@
 			)
 		)
-		(property "Footprint" ""
+		(property "Footprint" "payload_footprints:RESC1005X40N"
 			(at 88.646 65.024 90)
 			(hide yes)
@@
 			)
 		)
-		(property "Value" "C"
-			(at 197.866 71.374 90)
+		(property "Value" "100nF"
+			(at 200.152 71.374 90)
 			(show_name no)
 			(do_not_autoplace no)
@@
 			)
 		)
-		(property "Footprint" ""
+		(property "Footprint" "payload_footprints:CAPC1005X55N"
 			(at 199.39 71.4248 0)
 			(hide yes)
@@
 			)
 		)
-		(property "Value" "R_US"
+		(property "Value" "49.9K"
 			(at 110.49 66.0399 0)
 			(show_name no)
@@
 			)
 		)
-		(property "Footprint" ""
+		(property "Footprint" "payload_footprints:RESC1005X40N"
 			(at 108.966 65.024 90)
 			(hide yes)
@@
 			)
 		)
-		(property "Value" "C"
-			(at 197.866 119.634 90)
+		(property "Value" "100nF"
+			(at 200.152 119.634 90)
 			(show_name no)
 			(do_not_autoplace no)
@@
 			)
 		)
-		(property "Footprint" ""
+		(property "Footprint" "payload_footprints:CAPC1005X55N"
 			(at 199.39 119.6848 0)
 			(hide yes)
@@
 			)
 		)
-		(property "Value" "R_US"
+		(property "Value" "49.9K"
 			(at 82.55 66.0399 0)
 			(show_name no)
@@
 			)
 		)
-		(property "Footprint" ""
+		(property "Footprint" "payload_footprints:RESC1005X40N"
 			(at 81.026 65.024 90)
 			(hide yes)
@@
 			)
 		)
-		(property "Value" "C"
-			(at 197.866 114.554 90)
+		(property "Value" "100nF"
+			(at 200.152 114.554 90)
 			(show_name no)
 			(do_not_autoplace no)
@@
 			)
 		)
-		(property "Footprint" ""
+		(property "Footprint" "payload_footprints:CAPC1005X55N"
 			(at 199.39 114.6048 0)
 			(hide yes)
@@
 			)
 		)
-		(property "Value" "C"
-			(at 197.866 91.694 90)
+		(property "Value" "4.7uF"
+			(at 200.152 91.694 90)
 			(show_name no)
 			(do_not_autoplace no)
@@
 			)
 		)
-		(property "Footprint" ""
+		(property "Footprint" "payload_footprints:CAPC1608X90N"
 			(at 199.39 91.7448 0)
 			(hide yes)
@@
 			)
 		)
-		(property "Value" "C"
-			(at 197.866 81.534 90)
+		(property "Value" "100nF"
+			(at 200.152 81.534 90)
 			(show_name no)
 			(do_not_autoplace no)
@@
 			)
 		)
-		(property "Footprint" ""
+		(property "Footprint" "payload_footprints:CAPC1005X55N"
 			(at 199.39 81.5848 0)
 			(hide yes)
@@
 			)
 		)
-		(property "Value" "C"
-			(at 197.866 104.394 90)
+		(property "Value" "100nF"
+			(at 200.152 104.394 90)
 			(show_name no)
 			(do_not_autoplace no)
@@
 			)
 		)
-		(property "Footprint" ""
+		(property "Footprint" "payload_footprints:CAPC1005X55N"
 			(at 199.39 104.4448 0)
 			(hide yes)
@@
 			)
 		)
-		(property "Value" "R_US"
+		(property "Value" "49.9K"
 			(at 132.08 66.0399 0)
 			(show_name no)
@@
 			)
 		)
-		(property "Footprint" ""
+		(property "Footprint" "payload_footprints:RESC1005X40N"
 			(at 130.556 65.024 90)
 			(hide yes)
@@
 			)
 		)
-		(property "Value" "C"
-			(at 197.866 124.714 90)
+		(property "Value" "100nF"
+			(at 200.152 124.714 90)
 			(show_name no)
 			(do_not_autoplace no)
@@
 			)
 		)
-		(property "Footprint" ""
+		(property "Footprint" "payload_footprints:CAPC1005X55N"
 			(at 199.39 124.7648 0)
 			(hide yes)
@@
 			)
 		)
-		(property "Value" "R_US"
+		(property "Value" "10K"
 			(at 138.43 66.0399 0)
 			(show_name no)
@@
 			)
 		)
-		(property "Footprint" ""
+		(property "Footprint" "payload_footprints:RC0402N_YAG"
 			(at 136.906 65.024 90)
 			(hide yes)
@@
 			)
 		)
-		(property "Value" "C"
-			(at 197.866 86.614 90)
+		(property "Value" "100nF"
+			(at 200.152 86.614 90)
 			(show_name no)
 			(do_not_autoplace no)
@@
 			)
 		)
-		(property "Footprint" ""
+		(property "Footprint" "payload_footprints:CAPC1005X55N"
 			(at 199.39 86.6648 0)
 			(hide yes)
@@
 			)
 		)
-		(property "Value" "R_US"
+		(property "Value" "49.9K"
 			(at 104.14 66.0399 0)
 			(show_name no)
@@
 			)
 		)
-		(property "Footprint" ""
+		(property "Footprint" "payload_footprints:RESC1005X40N"
 			(at 102.616 65.024 90)
 			(hide yes)
@@
 			)
 		)
-		(property "Value" "R_US"
+		(property "Value" "49.9K"
 			(at 124.46 66.0399 0)
 			(show_name no)
@@
 			)
 		)
-		(property "Footprint" ""
+		(property "Footprint" "payload_footprints:RESC1005X40N"
 			(at 122.936 65.024 90)
 			(hide yes)
@@
 			)
 		)
-		(property "Value" "C"
-			(at 197.866 129.794 90)
+		(property "Value" "4.7uF"
+			(at 200.406 129.794 90)
 			(show_name no)
 			(do_not_autoplace no)
@@
 			)
 		)
-		(property "Footprint" ""
+		(property "Footprint" "payload_footprints:CAPC1608X90N"
 			(at 199.39 129.8448 0)
 			(hide yes)
@@
 			)
 		)
-		(property "Value" "C"
-			(at 197.866 109.474 90)
+		(property "Value" "100nF"
+			(at 200.152 109.474 90)
 			(show_name no)
 			(do_not_autoplace no)
@@
 			)
 		)
-		(property "Footprint" ""
+		(property "Footprint" "payload_footprints:CAPC1005X55N"
 			(at 199.39 109.5248 0)
 			(hide yes)
@@
 			)
 		)
-		(property "Value" "R_US"
+		(property "Value" "10K"
 			(at 146.05 66.0399 0)
 			(show_name no)
@@
 			)
 		)
-		(property "Footprint" ""
+		(property "Footprint" "payload_footprints:RC0402N_YAG"
 			(at 144.526 65.024 90)
 			(hide yes)
@@
 			)
 		)
-		(property "Value" "R_US"
+		(property "Value" "10K"
 			(at 118.11 113.0299 0)
 			(show_name no)
@@
 			)
 		)
-		(property "Footprint" ""
+		(property "Footprint" "payload_footprints:RC0402N_YAG"
 			(at 116.586 112.014 90)
 			(hide yes)
@@
 			)
 		)
-		(property "Value" "C"
-			(at 197.866 138.684 90)
+		(property "Value" "100nF"
+			(at 200.152 138.684 90)
 			(show_name no)
 			(do_not_autoplace no)
@@
 			)
 		)
-		(property "Footprint" ""
+		(property "Footprint" "payload_footprints:CAPC1005X55N"
 			(at 199.39 138.7348 0)
 			(hide yes)
@@
 			)
 		)
-		(property "Value" "C"
-			(at 197.866 76.454 90)
+		(property "Value" "100nF"
+			(at 200.152 76.454 90)
 			(show_name no)
 			(do_not_autoplace no)
@@
 			)
 		)
-		(property "Footprint" ""
+		(property "Footprint" "payload_footprints:CAPC1005X55N"
 			(at 199.39 76.5048 0)
 			(hide yes)
@@
 			)
 		)
-		(property "Value" "R_US"
+		(property "Value" "49.9K"
 			(at 96.52 66.0399 0)
 			(show_name no)
@@
 			)
 		)
-		(property "Footprint" ""
+		(property "Footprint" "payload_footprints:RESC1005X40N"
 			(at 94.996 65.024 90)
 			(hide yes)
