File: hardware/level_translators.kicad_sch (KiCad schematic)
At the start: 30 parts, among them U10 UM3304, U11 UM3304, U12 UM3304, U13 UM3304, U15 UM3304, U17 UM3304

Commit message: adding footprints to resistors and capacitors
Parts:
- R108, R111, R113, R115, R119, R143: value R_US -> 1M; footprint (none) -> payload_footprints:RC0402N_YAG
Changed lines of the file:
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@@
 			)
 		)
-		(property "Value" "R_US"
+		(property "Value" "1M"
 			(at 111.125 86.3599 0)
 			(show_name no)
@@
 			)
 		)
-		(property "Footprint" ""
+		(property "Footprint" "payload_footprints:RC0402N_YAG"
 			(at 108.204 84.836 90)
 			(hide yes)
@@
 			)
 		)
-		(property "Value" "R_US"
+		(property "Value" "1M"
 			(at 281.305 204.4699 0)
 			(show_name no)
@@
 			)
 		)
-		(property "Footprint" ""
+		(property "Footprint" "payload_footprints:RC0402N_YAG"
 			(at 278.384 202.946 90)
 			(hide yes)
@@
 			)
 		)
-		(property "Value" "R_US"
+		(property "Value" "1M"
 			(at 112.395 204.4699 0)
 			(show_name no)
@@
 			)
 		)
-		(property "Footprint" ""
+		(property "Footprint" "payload_footprints:RC0402N_YAG"
 			(at 109.474 202.946 90)
 			(hide yes)
@@
 			)
 		)
-		(property "Value" "R_US"
+		(property "Value" "1M"
 			(at 282.575 86.3599 0)
 			(show_name no)
@@
 			)
 		)
-		(property "Footprint" ""
+		(property "Footprint" "payload_footprints:RC0402N_YAG"
 			(at 279.654 84.836 90)
 			(hide yes)
@@
 			)
 		)
-		(property "Value" "R_US"
+		(property "Value" "1M"
 			(at 112.395 147.3199 0)
 			(show_name no)
@@
 			)
 		)
-		(property "Footprint" ""
+		(property "Footprint" "payload_footprints:RC0402N_YAG"
 			(at 109.474 145.796 90)
 			(hide yes)
@@
 			)
 		)
-		(property "Value" "R_US"
+		(property "Value" "1M"
 			(at 282.575 147.3199 0)
 			(show_name no)
@@
 			)
 		)
-		(property "Footprint" ""
+		(property "Footprint" "payload_footprints:RC0402N_YAG"
 			(at 279.654 145.796 90)
 			(hide yes)

Commit message: assigned footprints of resistors and some capacitors
Parts:
- C153, C155, C157, C159, C161, C163, C165, C167, C173, C175, C252, C253: value C -> 100nF; footprint (none) -> payload_footprints:CAP_CC0402_YAG
- R109, R110, R112, R114, R118, R142: value R_US -> 10K; footprint (none) -> payload_footprints:RC0402N_YAG
Changed lines of the file:
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@@
 			)
 		)
-		(property "Value" "C"
-			(at 248.158 194.056 90)
+		(property "Value" "100nF"
+			(at 251.714 194.056 90)
 			(show_name no)
 			(do_not_autoplace no)
@@
 			)
 		)
-		(property "Footprint" ""
+		(property "Footprint" "payload_footprints:CAP_CC0402_YAG"
 			(at 240.03 196.5452 0)
 			(hide yes)
@@
 			)
 		)
-		(property "Value" "R_US"
+		(property "Value" "10K"
 			(at 97.79 83.312 90)
 			(show_name no)
@@
 			)
 		)
-		(property "Footprint" ""
+		(property "Footprint" "payload_footprints:RC0402N_YAG"
 			(at 91.694 84.074 90)
 			(hide yes)
@@
 			)
 		)
-		(property "Value" "R_US"
+		(property "Value" "10K"
 			(at 269.24 83.312 90)
 			(show_name no)
@@
 			)
 		)
-		(property "Footprint" ""
+		(property "Footprint" "payload_footprints:RC0402N_YAG"
 			(at 263.144 84.074 90)
 			(hide yes)
@@
 			)
 		)
-		(property "Value" "R_US"
+		(property "Value" "10K"
 			(at 267.97 201.422 90)
 			(show_name no)
@@
 			)
 		)
-		(property "Footprint" ""
+		(property "Footprint" "payload_footprints:RC0402N_YAG"
 			(at 261.874 202.184 90)
 			(hide yes)
@@
 			)
 		)
-		(property "Value" "C"
-			(at 351.282 194.056 90)
+		(property "Value" "100nF"
+			(at 347.726 194.056 90)
 			(show_name no)
 			(do_not_autoplace no)
@@
 			)
 		)
-		(property "Footprint" ""
+		(property "Footprint" "payload_footprints:CAP_CC0402_YAG"
 			(at 359.41 196.5452 0)
 			(hide yes)
@@
 			)
 		)
-		(property "Value" "R_US"
+		(property "Value" "10K"
 			(at 99.06 201.422 90)
 			(show_name no)
@@
 			)
 		)
-		(property "Footprint" ""
+		(property "Footprint" "payload_footprints:RC0402N_YAG"
 			(at 92.964 202.184 90)
 			(hide yes)
@@
 			)
 		)
-		(property "Value" "C"
-			(at 79.248 136.906 90)
+		(property "Value" "100nF"
+			(at 82.55 136.906 90)
 			(show_name no)
 			(do_not_autoplace no)
@@
 			)
 		)
-		(property "Footprint" ""
+		(property "Footprint" "payload_footprints:CAP_CC0402_YAG"
 			(at 71.12 139.3952 0)
 			(hide yes)
@@
 			)
 		)
-		(property "Value" "C"
-			(at 249.428 75.946 90)
+		(property "Value" "100nF"
+			(at 252.73 75.946 90)
 			(show_name no)
 			(do_not_autoplace no)
@@
 			)
 		)
-		(property "Footprint" ""
+		(property "Footprint" "payload_footprints:CAP_CC0402_YAG"
 			(at 241.3 78.4352 0)
 			(hide yes)
@@
 			)
 		)
-		(property "Value" "C"
-			(at 79.248 194.056 90)
+		(property "Value" "100nF"
+			(at 83.058 194.056 90)
 			(show_name no)
 			(do_not_autoplace no)
@@
 			)
 		)
-		(property "Footprint" ""
+		(property "Footprint" "payload_footprints:CAP_CC0402_YAG"
 			(at 71.12 196.5452 0)
 			(hide yes)
@@
 			)
 		)
-		(property "Value" "C"
-			(at 249.428 136.906 90)
+		(property "Value" "100nF"
+			(at 252.476 136.906 90)
 			(show_name no)
 			(do_not_autoplace no)
@@
 			)
 		)
-		(property "Footprint" ""
+		(property "Footprint" "payload_footprints:CAP_CC0402_YAG"
 			(at 241.3 139.3952 0)
 			(hide yes)
@@
 			)
 		)
-		(property "Value" "R_US"
+		(property "Value" "10K"
 			(at 99.06 144.272 90)
 			(show_name no)
@@
 			)
 		)
-		(property "Footprint" ""
+		(property "Footprint" "payload_footprints:RC0402N_YAG"
 			(at 92.964 145.034 90)
 			(hide yes)
@@
 			)
 		)
-		(property "Value" "C"
-			(at 182.372 194.056 90)
+		(property "Value" "100nF"
+			(at 179.324 194.056 90)
 			(show_name no)
 			(do_not_autoplace no)
@@
 			)
 		)
-		(property "Footprint" ""
+		(property "Footprint" "payload_footprints:CAP_CC0402_YAG"
 			(at 190.5 196.5452 0)
 			(hide yes)
@@
 			)
 		)
-		(property "Value" "C"
-			(at 181.102 75.946 90)
+		(property "Value" "100nF"
+			(at 177.8 75.946 90)
 			(show_name no)
 			(do_not_autoplace no)
@@
 			)
 		)
-		(property "Footprint" ""
+		(property "Footprint" "payload_footprints:CAP_CC0402_YAG"
 			(at 189.23 78.4352 0)
 			(hide yes)
@@
 			)
 		)
-		(property "Value" "C"
-			(at 182.372 136.906 90)
+		(property "Value" "100nF"
+			(at 179.07 136.906 90)
 			(show_name no)
 			(do_not_autoplace no)
@@
 			)
 		)
-		(property "Footprint" ""
+		(property "Footprint" "payload_footprints:CAP_CC0402_YAG"
 			(at 190.5 139.3952 0)
 			(hide yes)
@@
 			)
 		)
-		(property "Value" "R_US"
+		(property "Value" "10K"
 			(at 269.24 144.272 90)
 			(show_name no)
@@
 			)
 		)
-		(property "Footprint" ""
+		(property "Footprint" "payload_footprints:RC0402N_YAG"
 			(at 263.144 145.034 90)
 			(hide yes)
@@
 			)
 		)
-		(property "Value" "C"
-			(at 352.552 75.946 90)
+		(property "Value" "100nF"
+			(at 348.996 75.946 90)
 			(show_name no)
 			(do_not_autoplace no)
@@
 			)
 		)
-		(property "Footprint" ""
+		(property "Footprint" "payload_footprints:CAP_CC0402_YAG"
 			(at 360.68 78.4352 0)
 			(hide yes)
@@
 			)
 		)
-		(property "Value" "C"
-			(at 77.978 75.946 90)
+		(property "Value" "100nF"
+			(at 81.28 75.946 90)
 			(show_name no)
 			(do_not_autoplace no)
@@
 			)
 		)
-		(property "Footprint" ""
+		(property "Footprint" "payload_footprints:CAP_CC0402_YAG"
 			(at 69.85 78.4352 0)
 			(hide yes)
@@
 			)
 		)
-		(property "Value" "C"
-			(at 352.552 136.906 90)
+		(property "Value" "100nF"
+			(at 349.25 136.906 90)
 			(show_name no)
 			(do_not_autoplace no)
@@
 			)
 		)
-		(property "Footprint" ""
+		(property "Footprint" "payload_footprints:CAP_CC0402_YAG"
 			(at 360.68 139.3952 0)
 			(hide yes)
