File: hardware/interfaces.kicad_sch (KiCad schematic)
At the start: 5 parts, among them J3 SSQ-126-04-G-D, J4 SSQ-126-04-G-D, J5 FFC_HDGC_1x22_0.5K-DX-22PWB

Commit message: adding footprints to resistors and capacitors
Parts:
- R136: value R_US -> 0R; footprint (none) -> payload_footprints:RC0402N_YAG
Changed lines of the file:
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@@
 			)
 		)
-		(property "Value" "R_US"
+		(property "Value" "0R"
 			(at 271.526 90.932 90)
 			(show_name no)
@@
 			)
 		)
-		(property "Footprint" ""
+		(property "Footprint" "payload_footprints:RC0402N_YAG"
 			(at 266.954 91.694 90)
 			(hide yes)

Commit message: assigned footprints of resistors and some capacitors
Parts:
- C185: value C -> 100nF; footprint (none) -> payload_footprints:CAPC1005X55N
Changed lines of the file:
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@@
 			)
 		)
-		(property "Value" "C"
+		(property "Value" "100nF"
 			(at 269.24 123.1899 0)
 			(show_name no)
@@
 			)
 		)
-		(property "Footprint" ""
+		(property "Footprint" "payload_footprints:CAPC1005X55N"
 			(at 266.3952 125.73 0)
 			(hide yes)

Commit message: renamed and assigned some connections concerning FPGA banks, sensors, interfaces
Connections:
- net PL_I2C_SDA: now reaches J3.41 (H1_41)
- net PL_I2C_SLC: now reaches J3.43 (H1_43)
- net POWER_ENABLE: no longer names the net of J3.20 (H1_20)
Changed lines of the file:
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@@
-	(wire
-		(pts
-			(xy 67.31 77.47) (xy 76.2 77.47)
-		)
-		(stroke
-			(width 0)
-			(type default)
-		)
-	)
 	(wire
 		(pts
@@
 	(wire
 		(pts
+			(xy 40.64 105.41) (xy 31.75 105.41)
+		)
+		(stroke
+			(width 0)
+			(type default)
+		)
+	)
+	(wire
+		(pts
 			(xy 40.64 90.17) (xy 30.48 90.17)
 		)
@@
 	(wire
 		(pts
-			(xy 154.94 111.76) (xy 163.83 111.76)
+			(xy 40.64 107.95) (xy 31.75 107.95)
 		)
 		(stroke
@@
 		)
 	)
-	(label "POWER_ENABLE"
-		(at 76.2 77.47 0)
-		(effects
-			(font
-				(size 1.27 1.27)
-			)
-			(justify left bottom)
+	(label "PL_I2C_SLC"
+		(at 31.75 107.95 180)
+		(effects
+			(font
+				(size 1.27 1.27)
+			)
+			(justify right bottom)
 		)
 	)
@@
 		)
 	)
-	(label "PWR_4_5V"
-		(at 163.83 111.76 0)
-		(effects
-			(font
-				(size 1.27 1.27)
-			)
-			(justify left bottom)
-		)
-	)
+	(label "PL_I2C_SDA"
+		(at 31.75 105.41 180)
+		(effects
+			(font
+				(size 1.27 1.27)
+			)
+			(justify right bottom)
+		)
+	)
