File: hardware/communication.kicad_sch (KiCad schematic)
At the start: 44 parts, among them IC10 TCA9517DGKRQ1, IC15 W25Q128JVSIQ, IC9 TCA9517DGKRQ1, U16 MPFS025T-FCVG484E, U8 SN65HVD234QDRQ1

Commit message: assigned footprints of resistors and some capacitors
Parts:
- C181: value C -> 100pF; footprint (none) -> payload_footprints:CAPC1005X55N
- C183: value C -> 100nF; footprint (none) -> payload_footprints:CAPC1005X55N
- R121, R124, R125, R132: value R_US -> 22R; footprint (none) -> payload_footprints:RC0402N_YAG
- R122, R126, R127, R128, R129, R130, R131, R133: value R_US -> 10K; footprint (none) -> payload_footprints:RC0402N_YAG
- R123: value R_US -> 1K; footprint (none) -> payload_footprints:RC0402N_YAG
Changed lines of the file:
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@@
 			)
 		)
-		(property "Value" "R_US"
+		(property "Value" "10K"
 			(at 256.286 43.434 0)
 			(show_name no)
@@
 			)
 		)
-		(property "Footprint" ""
+		(property "Footprint" "payload_footprints:RC0402N_YAG"
 			(at 263.906 43.434 90)
 			(hide yes)
@@
 			)
 		)
-		(property "Value" "R_US"
+		(property "Value" "10K"
 			(at 167.64 40.6399 0)
 			(show_name no)
@@
 			)
 		)
-		(property "Footprint" ""
+		(property "Footprint" "payload_footprints:RC0402N_YAG"
 			(at 166.116 39.624 90)
 			(hide yes)
@@
 			)
 		)
-		(property "Value" "R_US"
+		(property "Value" "1K"
 			(at 181.61 83.8199 0)
 			(show_name no)
@@
 			)
 		)
-		(property "Footprint" ""
+		(property "Footprint" "payload_footprints:RC0402N_YAG"
 			(at 180.086 82.804 90)
 			(hide yes)
@@
 			)
 		)
-		(property "Value" "R_US"
+		(property "Value" "22R"
 			(at 256.032 65.532 90)
 			(show_name no)
@@
 			)
 		)
-		(property "Footprint" ""
+		(property "Footprint" "payload_footprints:RC0402N_YAG"
 			(at 251.206 68.326 90)
 			(hide yes)
@@
 			)
 		)
-		(property "Value" "C"
+		(property "Value" "100pF"
 			(at 166.116 84.836 0)
 			(show_name no)
@@
 			)
 		)
-		(property "Footprint" ""
+		(property "Footprint" "payload_footprints:CAPC1005X55N"
 			(at 164.1348 78.74 0)
 			(hide yes)
@@
 			)
 		)
-		(property "Value" "R_US"
+		(property "Value" "10K"
 			(at 260.35 135.8899 0)
 			(show_name no)
@@
 			)
 		)
-		(property "Footprint" ""
+		(property "Footprint" "payload_footprints:RC0402N_YAG"
 			(at 258.826 134.874 90)
 			(hide yes)
@@
 			)
 		)
-		(property "Value" "R_US"
+		(property "Value" "10K"
 			(at 248.666 44.196 0)
 			(show_name no)
@@
 			)
 		)
-		(property "Footprint" ""
+		(property "Footprint" "payload_footprints:RC0402N_YAG"
 			(at 256.286 43.434 90)
 			(hide yes)
@@
 			)
 		)
-		(property "Value" "R_US"
+		(property "Value" "22R"
 			(at 183.388 65.278 90)
 			(show_name no)
@@
 			)
 		)
-		(property "Footprint" ""
+		(property "Footprint" "payload_footprints:RC0402N_YAG"
 			(at 178.816 68.326 90)
 			(hide yes)
@@
 			)
 		)
-		(property "Value" "R_US"
+		(property "Value" "10K"
 			(at 241.046 44.196 0)
 			(show_name no)
@@
 			)
 		)
-		(property "Footprint" ""
+		(property "Footprint" "payload_footprints:RC0402N_YAG"
 			(at 248.666 43.434 90)
 			(hide yes)
@@
 			)
 		)
-		(property "Value" "R_US"
+		(property "Value" "10K"
 			(at 177.8 138.4299 0)
 			(show_name no)
@@
 			)
 		)
-		(property "Footprint" ""
+		(property "Footprint" "payload_footprints:RC0402N_YAG"
 			(at 176.276 137.414 90)
 			(hide yes)
@@
 			)
 		)
-		(property "Value" "R_US"
+		(property "Value" "22R"
 			(at 241.808 146.558 90)
 			(show_name no)
@@
 			)
 		)
-		(property "Footprint" ""
+		(property "Footprint" "payload_footprints:RC0402N_YAG"
 			(at 237.236 149.606 90)
 			(hide yes)
@@
 			)
 		)
-		(property "Value" "R_US"
+		(property "Value" "10K"
 			(at 251.46 135.8899 0)
 			(show_name no)
@@
 			)
 		)
-		(property "Footprint" ""
+		(property "Footprint" "payload_footprints:RC0402N_YAG"
 			(at 249.936 134.874 90)
 			(hide yes)
@@
 			)
 		)
-		(property "Value" "R_US"
+		(property "Value" "10K"
 			(at 153.67 83.8199 0)
 			(show_name no)
@@
 			)
 		)
-		(property "Footprint" ""
+		(property "Footprint" "payload_footprints:RC0402N_YAG"
 			(at 152.146 82.804 90)
 			(hide yes)
@@
 			)
 		)
-		(property "Value" "C"
+		(property "Value" "100nF"
 			(at 228.346 135.636 0)
 			(show_name no)
@@
 			)
 		)
-		(property "Footprint" ""
+		(property "Footprint" "payload_footprints:CAPC1005X55N"
 			(at 226.3648 129.54 0)
 			(hide yes)
@@
 			)
 		)
-		(property "Value" "R_US"
+		(property "Value" "22R"
 			(at 256.286 61.722 90)
 			(show_name no)
@@
 			)
 		)
-		(property "Footprint" ""
+		(property "Footprint" "payload_footprints:RC0402N_YAG"
 			(at 251.206 64.516 90)
 			(hide yes)

Commit message: added USB components, updated BOM, marked components that still needs references
Changed lines of the file:
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@@
 	(generator_version "10.0")
 	(paper "A3")
+	(rectangle
+		(start 327.66 109.22)
+		(end 392.43 236.22)
+		(stroke
+			(width 0)
+			(type default)
+		)
+		(fill
+			(type none)
+		)
+	)
+	(rectangle
+		(start 20.32 19.05)
+		(end 115.57 276.86)
+		(stroke
+			(width 0)
+			(type default)
+		)
+		(fill
+			(type none)
+		)
+	)
 	(text "PROGRAMING THE SPI FLASH\nUSING EXTERNAL MASTER\n"
 		(exclude_from_sim no)
