File: hardware/fpga_power_banks.kicad_sch (KiCad schematic)
At the start: 86 parts, among them U4 MPFS025T-FCVG484E

Commit message: assigned footprints of resistors and some capacitors
Parts:
- C180, C190, C214, C216, C229, C236, C237, C241, C242, C245, C251: value C -> 47uF; footprint (none) -> payload_footprints:CAPC2012X145N
- C195, C199, C204, C208, C213, C219, C222: value C -> 10uF; footprint (none) -> payload_footprints:CAPC1608X100N
- R107: value R_US -> 10K; footprint (none) -> payload_footprints:RC0402N_YAG
Connections:
- net VCC_1V8: now also C217.2, C218.2, C219.2
- net VCC_2V5: no longer C217.2, C218.2, C219.2
Changed lines of the file:
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@@
 			)
 		)
-		(property "Value" "C"
+		(property "Value" "47uF"
 			(at 125.476 262.636 0)
 			(show_name no)
@@
 			)
 		)
-		(property "Footprint" ""
+		(property "Footprint" "payload_footprints:CAPC2012X145N"
 			(at 123.4948 256.54 0)
 			(hide yes)
@@
 			)
 		)
-		(property "Value" "C"
+		(property "Value" "47uF"
 			(at 89.916 262.636 0)
 			(show_name no)
@@
 			)
 		)
-		(property "Footprint" ""
+		(property "Footprint" "payload_footprints:CAPC2012X145N"
 			(at 87.9348 256.54 0)
 			(hide yes)
@@
 			)
 		)
-		(property "Value" "C"
+		(property "Value" "47uF"
 			(at 211.836 262.636 0)
 			(show_name no)
@@
 			)
 		)
-		(property "Footprint" ""
+		(property "Footprint" "payload_footprints:CAPC2012X145N"
 			(at 209.8548 256.54 0)
 			(hide yes)
@@
 			)
 		)
-		(property "Value" "C"
+		(property "Value" "10uF"
 			(at 279.146 182.626 0)
 			(show_name no)
@@
 			)
 		)
-		(property "Footprint" ""
+		(property "Footprint" "payload_footprints:CAPC1608X100N"
 			(at 277.1648 176.53 0)
 			(hide yes)
@@
 			)
 		)
-		(property "Value" "C"
+		(property "Value" "47uF"
 			(at 195.326 182.626 0)
 			(show_name no)
@@
 			)
 		)
-		(property "Footprint" ""
+		(property "Footprint" "payload_footprints:CAPC2012X145N"
 			(at 193.3448 176.53 0)
 			(hide yes)
@@
 			)
 		)
-		(property "Value" "C"
+		(property "Value" "10uF"
 			(at 166.116 221.996 0)
 			(show_name no)
@@
 			)
 		)
-		(property "Footprint" ""
+		(property "Footprint" "payload_footprints:CAPC1608X100N"
 			(at 164.1348 215.9 0)
 			(hide yes)
@@
 			)
 		)
-		(property "Value" "C"
+		(property "Value" "10uF"
 			(at 221.996 221.996 0)
 			(show_name no)
@@
 			)
 		)
-		(property "Footprint" ""
+		(property "Footprint" "payload_footprints:CAPC1608X100N"
 			(at 220.0148 215.9 0)
 			(hide yes)
@@
 		(in_pos_files yes)
 		(dnp no)
-		(fields_autoplaced yes)
 		(property "Reference" "#PWR0208"
 			(at 177.8 210.82 0)
@@
 			)
 		)
-		(property "Value" "VCC_2V5"
-			(at 177.8 201.93 0)
+		(property "Value" "VCC_1V8"
+			(at 173.99 201.93 0)
 			(show_name no)
 			(do_not_autoplace no)
@@
 					(size 1.27 1.27)
 				)
+				(justify left)
 			)
 		)
@@
 			)
 		)
-		(property "Value" "C"
+		(property "Value" "47uF"
 			(at 82.296 262.636 0)
 			(show_name no)
@@
 			)
 		)
-		(property "Footprint" ""
+		(property "Footprint" "payload_footprints:CAPC2012X145N"
 			(at 80.3148 256.54 0)
 			(hide yes)
@@
 			)
 		)
-		(property "Value" "C"
+		(property "Value" "10uF"
 			(at 138.176 221.996 0)
 			(show_name no)
@@
 			)
 		)
-		(property "Footprint" ""
+		(property "Footprint" "payload_footprints:CAPC1608X100N"
 			(at 136.1948 215.9 0)
 			(hide yes)
@@
 			)
 		)
-		(property "Value" "C"
+		(property "Value" "10uF"
 			(at 251.206 182.626 0)
 			(show_name no)
@@
 			)
 		)
-		(property "Footprint" ""
+		(property "Footprint" "payload_footprints:CAPC1608X100N"
 			(at 249.2248 176.53 0)
 			(hide yes)
@@
 			)
 		)
-		(property "Value" "C"
+		(property "Value" "47uF"
 			(at 144.526 182.626 0)
 			(show_name no)
@@
 			)
 		)
-		(property "Footprint" ""
+		(property "Footprint" "payload_footprints:CAPC2012X145N"
 			(at 142.5448 176.53 0)
 			(hide yes)
@@
 			)
 		)
-		(property "Value" "C"
+		(property "Value" "47uF"
 			(at 161.036 262.636 0)
 			(show_name no)
@@
 			)
 		)
-		(property "Footprint" ""
+		(property "Footprint" "payload_footprints:CAPC2012X145N"
 			(at 159.0548 256.54 0)
 			(hide yes)
@@
 			)
 		)
-		(property "Value" "C"
+		(property "Value" "47uF"
 			(at 280.416 221.996 0)
 			(show_name no)
@@
 			)
 		)
-		(property "Footprint" ""
+		(property "Footprint" "payload_footprints:CAPC2012X145N"
 			(at 278.4348 215.9 0)
 			(hide yes)
@@
 			)
 		)
-		(property "Value" "R_US"
+		(property "Value" "10K"
 			(at 206.375 113.0299 0)
 			(show_name no)
@@
 			)
 		)
-		(property "Footprint" ""
+		(property "Footprint" "payload_footprints:RC0402N_YAG"
 			(at 203.454 111.506 90)
 			(hide yes)
@@
 			)
 		)
-		(property "Value" "C"
+		(property "Value" "10uF"
 			(at 194.056 221.996 0)
 			(show_name no)
@@
 			)
 		)
-		(property "Footprint" ""
+		(property "Footprint" "payload_footprints:CAPC1608X100N"
 			(at 192.0748 215.9 0)
 			(hide yes)
@@
 			)
 		)
-		(property "Value" "C"
+		(property "Value" "47uF"
 			(at 133.096 262.636 0)
 			(show_name no)
@@
 			)
 		)
-		(property "Footprint" ""
+		(property "Footprint" "payload_footprints:CAPC2012X145N"
 			(at 131.1148 256.54 0)
 			(hide yes)
@@
 			)
 		)
-		(property "Value" "C"
+		(property "Value" "10uF"
 			(at 223.266 182.626 0)
 			(show_name no)
@@
 			)
 		)
-		(property "Footprint" ""
+		(property "Footprint" "payload_footprints:CAPC1608X100N"
 			(at 221.2848 176.53 0)
 			(hide yes)
@@
 			)
 		)
-		(property "Value" "C"
+		(property "Value" "47uF"
 			(at 110.236 221.996 0)
 			(show_name no)
@@
 			)
 		)
-		(property "Footprint" ""
+		(property "Footprint" "payload_footprints:CAPC2012X145N"
 			(at 108.2548 215.9 0)
 			(hide yes)
@@
 			)
 		)
-		(property "Value" "C"
+		(property "Value" "47uF"
 			(at 67.056 221.996 0)
 			(show_name no)
@@
 			)
 		)
-		(property "Footprint" ""
+		(property "Footprint" "payload_footprints:CAPC2012X145N"
 			(at 65.0748 215.9 0)
 			(hide yes)

Commit message: added capacitors footprints
Parts:
- C168, C170, C172, C189, C193, C194, C197, C198, C201, C202, C205, C206, C207, C209, C210, C211, C212, C215, C217, C218, C220, C221, C227, C228, C234, C235, C240, C244, C249, C250: value C -> 100nF; footprint (none) -> payload_footprints:CAPC0603X35N
- C174, C176, C178: value C -> 1uF; footprint (none) -> payload_footprints:CAP_CC0201_YAG
- C182, C184: value C_Polarized_US -> 330uF; footprint (none) -> payload_footprints:T520B
- C188, C192, C196, C200, C223, C243, C246: value C -> 1nF; footprint (none) -> payload_footprints:YAG_CC0201_YAG
- C224: value C -> 3.3nF; footprint (none) -> payload_footprints:CAPC0603X33N
- C230, C231: value C -> 2.2nF; footprint (none) -> payload_footprints:CAPC0603X33N

Commit message: added USB components, updated BOM, marked components that still needs references
Changed lines of the file:
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@@
 	(generator_version "10.0")
 	(paper "A3")
+	(rectangle
+		(start 48.26 255.27)
+		(end 63.5 265.43)
+		(stroke
+			(width 0)
+			(type default)
+		)
+		(fill
+			(type none)
+		)
+	)
+	(rectangle
+		(start 176.53 256.54)
+		(end 191.77 265.43)
+		(stroke
+			(width 0)
+			(type default)
+		)
+		(fill
+			(type none)
+		)
+	)
+	(rectangle
+		(start 40.64 214.63)
+		(end 48.26 223.52)
+		(stroke
+			(width 0)
+			(type default)
+		)
+		(fill
+			(type none)
+		)
+	)
+	(rectangle
+		(start 83.82 215.9)
+		(end 91.44 223.52)
+		(stroke
+			(width 0)
+			(type default)
+		)
+		(fill
+			(type none)
+		)
+	)
+	(rectangle
+		(start 245.11 215.9)
+		(end 261.62 224.79)
+		(stroke
+			(width 0)
+			(type default)
+		)
+		(fill
+			(type none)
+		)
+	)
+	(rectangle
+		(start 97.79 255.27)
+		(end 113.03 264.16)
+		(stroke
+			(width 0)
+			(type default)
+		)
+		(fill
+			(type none)
+		)
+	)
+	(rectangle
+		(start 33.02 173.99)
+		(end 95.25 185.42)
+		(stroke
+			(width 0)
+			(type default)
+		)
+		(fill
+			(type none)
+		)
+	)
+	(rectangle
+		(start 167.64 176.53)
+		(end 184.15 184.15)
+		(stroke
+			(width 0)
+			(type default)
+		)
+		(fill
+			(type none)
+		)
+	)
 	(text "POWER BANKS"
 		(exclude_from_sim no)
