File: hardware/max2771.kicad_sch (KiCad schematic)
At the start: 50 parts, among them IC16 MAX8510EXK29+T, IC17 MAX8510EXK29+T, IC7 MAX2771ETI+, J6 Conn_Coaxial

Commit message: renamed and assigned some connections concerning FPGA banks, sensors, interfaces
Other:
- note added: "I/Q SIGNALS TEST POINTS"
- note removed: "PROGRAMING THE SPI FLASH USING EXTERNAL MASTER"
Changed lines of the file:
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@@
 	(generator_version "10.0")
 	(paper "A3")
-	(text "PROGRAMING THE SPI FLASH\nUSING EXTERNAL MASTER\n"
+	(text "I/Q SIGNALS TEST POINTS"
 		(exclude_from_sim no)
 		(at 371.094 31.496 0)

Commit message: added USB components, updated BOM, marked components that still needs references
Changed lines of the file:
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@@
 	(generator_version "10.0")
 	(paper "A3")
+	(rectangle
+		(start 20.32 15.24)
+		(end 402.59 260.35)
+		(stroke
+			(width 0)
+			(type default)
+		)
+		(fill
+			(type none)
+		)
+	)
 	(text "I/Q SIGNALS TEST POINTS"
 		(exclude_from_sim no)
