File: hardware/power_supply.kicad_sch (KiCad schematic)
At the start: 122 parts, among them IC1 MIC5504-2.5YM5-TR, IC2 TLV62569DBVT, IC3 MIC23303YML-TR, IC4 MIC23303YML-TR, IC5 MIC23303YML-TR, J1 Conn_01x02, Q1 RQ3E120ATTB, Q2 MMBT3906LT3G, Q3 RQ3E120ATTB, Q4 RQ3E120ATTB, Q5 BCM857BS-7-F, Q6 RQ3E120ATTB, Q7 BCM857BS-7-F, Q8 BCM857BS-7-F, Q9 BCM857BS-7-F, U1 ATL431AIDBZR, U2 MIC22950YML-TR, U3 MCP1725T-ADJE/MC

Commit message: adding footprints to resistors and capacitors
Parts:
- R24, R27: value R_US -> 0R; footprint (none) -> payload_footprints:RC0402N_YAG
- R8: value R_US -> 1M; footprint (none) -> payload_footprints:RC0402N_YAG
Changed lines of the file:
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@@
 		(color 0 0 0 0)
 	)
-	(bus_entry
-		(at 236.22 96.52)
-		(size 2.54 2.54)
-		(stroke
-			(width 0)
-			(type default)
-		)
-	)
 	(wire
 		(pts
@@
 			)
 		)
-		(property "Value" "R_US"
+		(property "Value" "0R"
 			(at 274.32 186.69 90)
 			(show_name no)
@@
 			)
 		)
-		(property "Footprint" ""
+		(property "Footprint" "payload_footprints:RC0402N_YAG"
 			(at 274.574 189.484 90)
 			(hide yes)
@@
 			)
 		)
-		(property "Value" "R_US"
+		(property "Value" "1M"
 			(at 137.16 48.26 90)
 			(show_name no)
@@
 			)
 		)
-		(property "Footprint" ""
+		(property "Footprint" "payload_footprints:RC0402N_YAG"
 			(at 137.414 51.054 90)
 			(hide yes)
@@
 			)
 		)
-		(property "Value" "R_US"
+		(property "Value" "0R"
 			(at 274.32 118.11 90)
 			(show_name no)
@@
 			)
 		)
-		(property "Footprint" ""
+		(property "Footprint" "payload_footprints:RC0402N_YAG"
 			(at 274.574 120.904 90)
 			(hide yes)

Commit message: assigned footprints of resistors and some capacitors
Parts:
- C11: value C -> 470pF; footprint (none) -> payload_footprints:CAPC1005X55N
- C17, C18: value C -> 47uF; footprint (none) -> payload_footprints:CAPC2012X145N
- C19, C22: value C -> 100pF; footprint (none) -> payload_footprints:CAPC1005X55N
- C2, C26, C30, C36, C44: value C -> 100nF; footprint (none) -> payload_footprints:CAPC1005X55N
- C20, C32, C40, C48: value C -> 33pF; footprint (none) -> payload_footprints:CAPC1005X55N
- C21: value C -> 10nF; footprint (none) -> payload_footprints:CAPC1005X55N
- C23, C29, C35, C43: value C -> 4.7uF; footprint (none) -> payload_footprints:CAPC2012X145N
- C31, C37, C4, C45, C5, C6, C8: value C -> 1uF; footprint (none) -> payload_footprints:YAG_CC0402_YAG
- C9: value C -> 10uF; footprint (none) -> payload_footprints:CAPC1608X100N
- R1: value R_US -> 51K; footprint (none) -> payload_footprints:RC0402N_PAN
- R10, R11, R12, R13: value R_US -> 49.9K; footprint (none) -> payload_footprints:RESC1005X40N
- R15, R22, R29, R34, R6: value R_US -> 10K; footprint (none) -> payload_footprints:RC0402N_YAG
- R16: value R_US -> 20K; footprint (none) -> payload_footprints:RESC1005X40N
- R18: value R_US -> 2.49K; footprint (none) -> payload_footprints:RESC1005X40N
- R19, R21, R26, R3, R5, R7: value R_US -> 100K; footprint (none) -> payload_footprints:RESC1005X40N
- R2: value R_US -> 2.7K; footprint (none) -> payload_footprints:RESC1005X40N
- R20: value R_US -> 200K; footprint (none) -> payload_footprints:RESC1005X40N
- R23, R28, R33: value R_US -> 10R; footprint (none) -> payload_footprints:RESC1005X40N
- R25: value R_US -> 432K; footprint (none) -> payload_footprints:RESC1005X40N
- R30: value R_US -> 240K; footprint (none) -> payload_footprints:RESC1005X40N
- R31: value R_US -> 124K; footprint (none) -> payload_footprints:RESC1005X40N
- R35: value R_US -> 82K; footprint (none) -> payload_footprints:RESC1005X40N
- R36: value R_US -> 105K; footprint (none) -> payload_footprints:RESC1005X40N
- R4: value R_US -> 2.2K; footprint (none) -> payload_footprints:RESC1005X40N
- R9: value R_US -> 1K; footprint (none) -> payload_footprints:RC0402N_YAG
Connections:
- net GNDREF: now also IC2.2 (GND)
Other:
- moved on the sheet: C18

Commit message: added capacitors footprints
Parts:
- C10, C14, C15, C16, C33, C34, C41, C42, C49, C50: value C -> 22uF; footprint (none) -> payload_footprints:CAPC2012X145N
- C12, C13: value C -> 1nF; footprint (none) -> payload_footprints:YAG_CC0402_YAG
- C24: value C -> 6.8pF; footprint (none) -> payload_footprints:CAPC1005X70N
- C25: value C -> 22uF
- C7: value C -> 1uF; footprint (none) -> payload_footprints:YAG_CC0402_YAG
Changed lines of the file:
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@@
 			)
 		)
-		(property "Value" "C"
+		(property "Value" "1nF"
 			(at 66.04 267.9699 0)
 			(show_name no)
@@
 			)
 		)
-		(property "Footprint" ""
+		(property "Footprint" "payload_footprints:YAG_CC0402_YAG"
 			(at 63.1952 270.51 0)
 			(hide yes)
@@
 			)
 		)
-		(property "Value" "C"
+		(property "Value" "22uF"
 			(at 369.57 39.3699 0)
 			(show_name no)
@@
 			)
 		)
-		(property "Value" "C"
+		(property "Value" "22uF"
 			(at 50.8 215.8999 0)
 			(show_name no)
@@
 			)
 		)
-		(property "Footprint" ""
+		(property "Footprint" "payload_footprints:CAPC2012X145N"
 			(at 47.9552 218.44 0)
 			(hide yes)
@@
 			)
 		)
-		(property "Value" "C"
+		(property "Value" "22uF"
 			(at 391.16 93.9799 0)
 			(show_name no)
@@
 			)
 		)
-		(property "Footprint" ""
+		(property "Footprint" "payload_footprints:CAPC2012X145N"
 			(at 388.3152 96.52 0)
 			(hide yes)
@@
 			)
 		)
-		(property "Value" "C"
+		(property "Value" "22uF"
 			(at 382.27 227.3299 0)
 			(show_name no)
@@
 			)
 		)
-		(property "Footprint" ""
+		(property "Footprint" "payload_footprints:CAPC2012X145N"
 			(at 379.4252 229.87 0)
 			(hide yes)
@@
 			)
 		)
-		(property "Value" "C"
+		(property "Value" "22uF"
 			(at 370.84 227.3299 0)
 			(show_name no)
@@
 			)
 		)
-		(property "Footprint" ""
+		(property "Footprint" "payload_footprints:CAPC2012X145N"
 			(at 367.9952 229.87 0)
 			(hide yes)
@@
 			)
 		)
-		(property "Value" "C"
+		(property "Value" "6.8pF"
 			(at 354.33 39.3699 0)
 			(show_name no)
@@
 			)
 		)
-		(property "Footprint" ""
+		(property "Footprint" "payload_footprints:CAPC1005X70N"
 			(at 351.4852 41.91 0)
 			(hide yes)
@@
 			)
 		)
-		(property "Value" "C"
+		(property "Value" "22uF"
 			(at 391.16 162.5599 0)
 			(show_name no)
@@
 			)
 		)
-		(property "Footprint" ""
+		(property "Footprint" "payload_footprints:CAPC2012X145N"
 			(at 388.3152 165.1 0)
 			(hide yes)
@@
 			)
 		)
-		(property "Value" "C"
+		(property "Value" "1nF"
 			(at 55.88 267.9699 0)
 			(show_name no)
@@
 			)
 		)
-		(property "Footprint" ""
+		(property "Footprint" "payload_footprints:YAG_CC0402_YAG"
 			(at 53.0352 270.51 0)
 			(hide yes)
@@
 			)
 		)
-		(property "Value" "C"
+		(property "Value" "22uF"
 			(at 60.96 215.8999 0)
 			(show_name no)
@@
 			)
 		)
-		(property "Footprint" ""
+		(property "Footprint" "payload_footprints:CAPC2012X145N"
 			(at 58.1152 218.44 0)
 			(hide yes)
@@
 			)
 		)
-		(property "Value" "C"
+		(property "Value" "22uF"
 			(at 39.37 215.8999 0)
 			(show_name no)
@@
 			)
 		)
-		(property "Footprint" ""
+		(property "Footprint" "payload_footprints:CAPC2012X145N"
 			(at 36.5252 218.44 0)
 			(hide yes)
@@
 			)
 		)
-		(property "Value" "C"
+		(property "Value" "1uF"
 			(at 180.34 175.2599 0)
 			(show_name no)
@@
 			)
 		)
-		(property "Footprint" ""
+		(property "Footprint" "payload_footprints:YAG_CC0402_YAG"
 			(at 177.4952 177.8 0)
 			(hide yes)
@@
 			)
 		)
-		(property "Value" "C"
+		(property "Value" "22uF"
 			(at 379.73 93.9799 0)
 			(show_name no)
@@
 			)
 		)
-		(property "Footprint" ""
+		(property "Footprint" "payload_footprints:CAPC2012X145N"
 			(at 376.8852 96.52 0)
 			(hide yes)
@@
 			)
 		)
-		(property "Value" "C"
+		(property "Value" "22uF"
 			(at 379.73 162.5599 0)
 			(show_name no)
@@
 			)
 		)
-		(property "Footprint" ""
+		(property "Footprint" "payload_footprints:CAPC2012X145N"
 			(at 376.8852 165.1 0)
 			(hide yes)
@@
 			)
 		)
-		(property "Value" "C"
+		(property "Value" "22uF"
 			(at 27.94 215.8999 0)
 			(show_name no)
@@
 			)
 		)
-		(property "Footprint" ""
+		(property "Footprint" "payload_footprints:CAPC2012X145N"
 			(at 25.0952 218.44 0)
 			(hide yes)

Commit message: renamed and assigned some connections concerning FPGA banks, sensors, interfaces
Parts:
- removed J1: Conn_01x02, symbol Connector_Generic:Conn_01x02
Changed lines of the file:
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@@
 	(wire
 		(pts
-			(xy 36.83 30.48) (xy 38.1 30.48)
-		)
-		(stroke
-			(width 0)
-			(type default)
-		)
-	)
-	(wire
-		(pts
 			(xy 63.5 160.02) (xy 71.12 160.02)
 		)
@@
 	(wire
 		(pts
-			(xy 36.83 27.94) (xy 46.99 27.94)
+			(xy 256.54 207.01) (xy 256.54 215.9)
 		)
 		(stroke
@@
 	(wire
 		(pts
-			(xy 256.54 207.01) (xy 256.54 215.9)
+			(xy 350.52 31.75) (xy 339.09 31.75)
 		)
 		(stroke
@@
 	(wire
 		(pts
-			(xy 350.52 31.75) (xy 339.09 31.75)
+			(xy 153.67 213.36) (xy 153.67 207.01)
 		)
 		(stroke
@@
 	(wire
 		(pts
-			(xy 153.67 213.36) (xy 153.67 207.01)
+			(xy 30.48 30.48) (xy 38.1 30.48)
 		)
 		(stroke
@@
 	(wire
 		(pts
+			(xy 30.48 27.94) (xy 46.99 27.94)
+		)
+		(stroke
+			(width 0)
+			(type default)
+		)
+	)
+	(wire
+		(pts
 			(xy 336.55 82.55) (xy 344.17 82.55)
 		)
@@
 		)
 	)
+	(label "PWR_4_5V"
+		(at 30.48 27.94 180)
+		(effects
+			(font
+				(size 1.27 1.27)
+			)
+			(justify right bottom)
+		)
+	)
+	(label "GND"
+		(at 30.48 30.48 180)
+		(effects
+			(font
+				(size 1.27 1.27)
+			)
+			(justify right bottom)
+		)
+	)
 	(label "PG_1V"
 		(at 252.73 121.92 0)
@@
 					(unit 1)
 				)
-			)
-		)
-	)
-	(symbol
-		(lib_id "Connector_Generic:Conn_01x02")
-		(at 31.75 27.94 0)
-		(mirror y)
-		(unit 1)
-		(body_style 1)
-		(exclude_from_sim no)
-		(in_bom yes)
-		(on_board yes)
-		(in_pos_files yes)
-		(dnp no)
-		(fields_autoplaced yes)
-		(property "Reference" "J1"
-			(at 29.21 27.9399 0)
-			(show_name no)
-			(do_not_autoplace no)
-			(effects
-				(font
-					(size 1.27 1.27)
-				)
-				(justify left)
-			)
-		)
-		(property "Value" "Conn_01x02"
-			(at 29.21 30.4799 0)
-			(show_name no)
-			(do_not_autoplace no)
-			(effects
-				(font
-					(size 1.27 1.27)
-				)
-				(justify left)
-			)
-		)
-		(property "Footprint" ""
-			(at 31.75 27.94 0)
-			(hide yes)
-			(show_name no)
-			(do_not_autoplace no)
-			(effects
-				(font
-					(size 1.27 1.27)
-				)
-			)
-		)
-		(property "Datasheet" ""
-			(at 31.75 27.94 0)
-			(hide yes)
-			(show_name no)
-			(do_not_autoplace no)
-			(effects
-				(font
-					(size 1.27 1.27)
-				)
-			)
-		)
-		(property "Description" "Generic connector, single row, 01x02, script generated (kicad-library-utils/schlib/autogen/connector/)"
-			(at 31.75 27.94 0)
-			(hide yes)
-			(show_name no)
-			(do_not_autoplace no)
-			(effects
-				(font
-					(size 1.27 1.27)
-				)
-			)
-		)
-		(pin "2"
-		)
-		(pin "1"
-		)
-		(instances
-			(project "RO-Instrument"
-				(path "/1b019b3c-bb85-464b-9592-d957470b2156"
-					(reference "J1")
-					(unit 1)
-				)

Commit message: added USB components, updated BOM, marked components that still needs references
Changed lines of the file:
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@@
+	)
+	(rectangle
+		(start 297.18 173.99)
+		(end 312.42 181.61)
+		(stroke
+			(width 0)
+			(type default)
+		)
+		(fill
+			(type none)
+		)
+	)
+	(rectangle
+		(start 334.01 208.28)
+		(end 344.17 218.44)
+		(stroke
+			(width 0)
+			(type default)
+		)
+		(fill
+			(type none)
+		)
 	)
 	(rectangle
 		(start 95.25 137.16)
 		(end 223.52 191.77)
+		(stroke
+			(width 0)
+			(type default)
+		)
+		(fill
+			(type none)
+		)
+	)
+	(rectangle
+		(start 321.31 25.4)
+		(end 334.01 35.56)
+		(stroke
+			(width 0)
+			(type default)
+		)
+		(fill
+			(type none)
+		)
+	)
+	(rectangle
+		(start 167.64 45.72)
+		(end 180.34 54.61)
+		(stroke
+			(width 0)
+			(type default)
+		)
+		(fill
+			(type none)
+		)
+	)
+	(rectangle
+		(start 257.81 247.65)
+		(end 273.05 260.35)
+		(stroke
+			(width 0)
+			(type default)
+		)
+		(fill
+			(type none)
+		)
+	)
+	(rectangle
+		(start 288.29 193.04)
+		(end 303.53 200.66)
+		(stroke
+			(width 0)
+			(type default)
+		)
+		(fill
+			(type none)
+		)
+	)
+	(rectangle
+		(start 288.29 237.49)
+		(end 300.99 246.38)
+		(stroke
+			(width 0)
+			(type default)
+		)
+		(fill
+			(type none)
+		)
+	)
+	(rectangle
+		(start 344.17 73.66)
+		(end 353.06 85.09)
+		(stroke
+			(width 0)
+			(type default)
+		)
+		(fill
+			(type none)
+		)
+	)
+	(rectangle
+		(start 279.4 256.54)
+		(end 293.37 262.89)
+		(stroke
+			(width 0)
+			(type default)
+		)
+		(fill
+			(type none)
+		)
+	)
+	(rectangle
+		(start 297.18 104.14)
+		(end 311.15 111.76)
+		(stroke
+			(width 0)
+			(type default)
+		)
+		(fill
+			(type none)
+		)
+	)
+	(rectangle
+		(start 66.04 31.75)
+		(end 77.47 40.64)
 		(stroke
 			(width 0)
@@
 	)
 	(rectangle
+		(start 193.04 152.4)
+		(end 205.74 160.02)
+		(stroke
+			(width 0)
+			(type default)
+		)
+		(fill
+			(type none)
+		)
+	)
+	(rectangle
 		(start 15.24 15.24)
 		(end 223.52 137.16)
 		(stroke
 			(width 0)
+			(type default)
+		)
+		(fill
+			(type none)
+		)
+	)
+	(rectangle
+		(start 288.29 123.19)
+		(end 303.53 132.08)
+		(stroke
+			(width 0)
+			(type default)
+		)
+		(fill
+			(type none)
+		)
+	)
+	(rectangle
+		(start 344.17 142.24)
+		(end 353.06 154.94)
+		(stroke
+			(width 0)
+			(type default)
+		)
+		(fill
+			(type none)
+		)
+	)
+	(rectangle
+		(start 129.54 198.12)
+		(end 138.43 212.09)
+		(stroke
+			(width 0)

Commit message: assigned usb resistors and capacitors footprints, created a preliminary 3D PCB model
Other:
- moved on the sheet: TP5
Changed lines of the file:
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@@
 	(wire
 		(pts
-			(xy 167.64 207.01) (xy 171.45 207.01)
+			(xy 167.64 207.01) (xy 191.77 207.01)
 		)
 		(stroke
@@
 		)
 	)
+	(label "OUT_VCC_1V"
+		(at 172.72 207.01 0)
+		(effects
+			(font
+				(size 1.27 1.27)
+			)
+			(justify left bottom)
+		)
+	)
+	(label "OUT_VCC_2V5"
+		(at 73.66 160.02 0)
+		(effects
+			(font
+				(size 1.27 1.27)
+			)
+			(justify left bottom)
+		)
+	)
 	(label "PG_1V"
 		(at 252.73 190.5 0)
@@
 		)
 	)
+	(label "OUT_VCCA_1V"
+		(at 199.39 149.86 0)
+		(effects
+			(font
+				(size 1.27 1.27)
+			)
+			(justify left bottom)
+		)
+	)
+	(label "OUT_VCC_1V8"
+		(at 389.89 151.13 0)
+		(effects
+			(font
+				(size 1.27 1.27)
+			)
+			(justify left bottom)
+		)
+	)
+	(label "OUT_VCC_1V1"
+		(at 381 215.9 0)
+		(effects
+			(font
+				(size 1.27 1.27)
+			)
+			(justify left bottom)
+		)
+	)
 	(label "EXT_VDD_5V"
 		(at 40.64 27.94 0)
@@
 		)
 	)
+	(label "OUT_VCC_3V3"
+		(at 388.62 82.55 0)
+		(effects
+			(font
+				(size 1.27 1.27)
+			)
+			(justify left bottom)
+		)
+	)
 	(label "PG_1V"
 		(at 252.73 121.92 0)
@@
 		)
 	)
+	(label "OUT_VIO_ENABLE"
+		(at 379.73 31.75 0)
+		(effects
+			(font
+				(size 1.27 1.27)
+			)
+			(justify left bottom)
+		)
+	)
 	(symbol
 		(lib_id "power:VDD")
@@
 	(symbol
 		(lib_id "Connector:TestPoint")
-		(at 171.45 207.01 270)
+		(at 191.77 207.01 270)
 		(unit 1)
 		(body_style 1)
@@
 		(fields_autoplaced yes)
 		(property "Reference" "TP5"
-			(at 176.53 205.7399 90)
+			(at 196.85 205.7399 90)
 			(show_name no)
 			(do_not_autoplace no)
@@
 		)
 		(property "Value" "TestPoint"
-			(at 176.53 208.2799 90)
+			(at 196.85 208.2799 90)
 			(show_name no)
 			(do_not_autoplace no)
@@
 		)
 		(property "Footprint" ""
-			(at 171.45 212.09 0)
+			(at 191.77 212.09 0)
 			(hide yes)
 			(show_name no)
@@
 		)
 		(property "Datasheet" ""
-			(at 171.45 212.09 0)
+			(at 191.77 212.09 0)
 			(hide yes)
 			(show_name no)
@@
 		)
 		(property "Description" "test point"
-			(at 171.45 207.01 0)
+			(at 191.77 207.01 0)
 			(hide yes)
 			(show_name no)
