File: hardware/sensing.kicad_sch (KiCad schematic)
At the start: 20 parts, among them IC13 INA226AQDGSRQ1, IC14 TMP112AQDRLRQ1, IC18 INA226AQDGSRQ1, IC19 INA226AQDGSRQ1, IC20 INA226AQDGSRQ1, IC21 INA226AQDGSRQ1, IC22 INA226AQDGSRQ1

Commit message: added USB components, updated BOM, marked components that still needs references
Parts:
- added IC23, IC24, IC25, IC26, IC27, IC28, IC29: SI1416EDH-T1-GE3, SOT65P210X110-6N, symbol payload-sym:SI1416EDH-T1-GE3
- added U14, U18, U19, U20, U21, U22: LTC4361HDC-2-TRMPBF, DFN-8_DC_LIT, symbol payload-sym:LTC4361HDC-2-TRMPBF
Other:
- moved on the sheet: C177, C179, C261, IC13, IC14, IC18, R120, R150

Commit message: assigned usb resistors and capacitors footprints, created a preliminary 3D PCB model
Parts:
- removed C177: C, symbol Device:C
- removed IC14: TMP112AQDRLRQ1, SOTFL50P160X60-6N, symbol payload-sym:TMP112AQDRLRQ1
- removed IC23, IC24, IC25, IC26, IC27, IC29: SI1416EDH-T1-GE3, SOT65P210X110-6N, symbol payload-sym:SI1416EDH-T1-GE3
- removed U18, U19, U20, U21, U22: LTC4361HDC-2-TRMPBF, DFN-8_DC_LIT, symbol payload-sym:LTC4361HDC-2-TRMPBF
Connections:
- net SLA_I2C_SDA: now reaches IC22.4 (SDA)
- net SLA_I2C_SDA: now also IC13.4 (SDA), IC18.4 (SDA), IC19.4 (SDA), IC20.4 (SDA), IC21.4 (SDA)
- net SLA_I2C_SCL: now reaches IC22.5 (SCL)
- net SLA_I2C_SCL: now also IC13.5 (SCL), IC18.5 (SCL), IC19.5 (SCL), IC20.5 (SCL), IC21.5 (SCL)
Other:
- note removed: "TEMPERATURE SENSOR"
- moved on the sheet: C262, C263, C264, C265, IC19, IC20, IC21, IC22, IC28, R151, R152, R153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
